File: hardware/kicad/LoRa_Boat_Controller.kicad_sch (KiCad schematic)
At the start: 45 parts, among them U1 SB007-03Q-TL-E, U3 STM32F4XXR2, U5 TCAN1042H-Q1D, U6 R1240N001x

Commit message: Snapshot pre-reconstruction state before Phase A
Adds the untracked KiCad sub-sheets, stale pipeline docs (STATUS/SESSION_HANDOFF/DIRECTIVES),
the agent brief (AGENT_PROMPT_V2.md), and the legacy DSN converter that were left uncommitted
by the previous session. Nothing here is validated; it is captured so the reconstruction diff
is reviewable. .gitignore now excludes .claude/, *.lck, _backup_*/ and KiCad autosaves.

Co-Authored-By: Claude Fable 5.1 <noreply@anthropic.com>
Parts:
- removed C1, C2, C3, C4, C5, C6, C7, C8, C9: 100n, Capacitor_SMD:C_0402_1005Metric, symbol Device:C
- removed C10: 4.7uF, Capacitor_SMD:C_0603_1608Metric, symbol Device:C
- removed C12: .1uf, Capacitor_SMD:C_0603_1608Metric, symbol Device:C
- removed C14: 470pF, Capacitor_SMD:C_0603_1608Metric, symbol Device:C
- removed C20, C21: 10uF, Capacitor_SMD:C_0805_2012Metric, symbol Device:C
- removed C22: .1uF, Capacitor_SMD:C_0603_1608Metric, symbol Device:C
- removed C23: 47pF, Capacitor_SMD:C_0402_1005Metric, symbol Device:C
- removed CANHEADER: CONN_B4B-XH-A, Connector_JST:JST_XH_B4B-XH-A_1x04_P2.50mm_Vertical, symbol Device:C
- removed CEXT: 4.7 uF, Capacitor_SMD:C_0603_1608Metric, symbol Device:C
- removed CIN: 10uF, Capacitor_SMD:C_1210_3225Metric, symbol Device:C
- removed COUT, COUT1: 10uf, Capacitor_SMD:C_1206_3216Metric, symbol Device:C
- removed GND: Battery-, Connector_PinHeader_2.54mm:PinHeader_1x01_P2.54mm_Vertical, symbol Connector:Conn_01x01_Pin
- removed GPSMODULE: CONN5_1LFBN-RC, Connector_PinHeader_2.54mm:PinHeader_1x05_P2.54mm_Vertical, symbol Connector:Conn_01x05_Pin
- removed JTAG: CONN_010P_000C_1, Connector_IDC:IDC-Header_2x05_P2.54mm_Vertical, symbol Connector:Conn_02x05_Odd_Even
- removed L1: 4.7uH, Inductor_SMD:L_0603_1608Metric, symbol Device:L
- removed L3, L4: INDUCTOR, Inductor_SMD:L_0402_1005Metric, symbol Device:L
- removed LORAMODULE: CONN5_1LFBN-RC, Connector_PinHeader_2.54mm:PinHeader_1x05_P2.54mm_Vertical, symbol Device:L
- removed R1: 15K, Resistor_SMD:R_0402_1005Metric, symbol Device:R
- removed R2: 4.7K, Resistor_SMD:R_0603_1608Metric, symbol Device:R
- removed R3: 51, Resistor_SMD:R_0402_1005Metric, symbol Device:R
- removed R4: 5.1K, Resistor_SMD:R_0402_1005Metric, symbol Device:R
- removed R5: 30K, Resistor_SMD:R_0805_2012Metric, symbol Device:R
- removed R6: 10K, Resistor_SMD:R_0402_1005Metric, symbol Device:R
- removed SPEEDCONTROLLER, STEERINGSERVO: CONN_PPTC031, Connector_PinHeader_2.54mm:PinHeader_1x03_P2.54mm_Vertical, symbol Connector:Conn_01x03_Pin
- removed TP1, TP3, TP4, TP5: TEST POINT, TestPoint:TestPoint_Pad_D1.0mm, symbol Connector:TestPoint
- removed U1: SB007-03Q-TL-E, Package_TO_SOT_SMD:SOT-323_SC-70, symbol Device:D_Schottky
- removed U3: STM32F4XXR2, Package_QFP:LQFP-64_10x10mm_P0.5mm, symbol MCU_ST:STM32F446RETx
- removed U5: TCAN1042H-Q1D, Package_SO:SOIC-8_3.9x4.9mm_P1.27mm, symbol Interface_CAN_LIN:TCAN1042
- removed U6: R1240N001x, Package_TO_SOT_SMD:SOT-23-6, symbol Regulator_Switching:R1240N001x
- removed VIN: Battery+, Connector_PinHeader_2.54mm:PinHeader_1x01_P2.54mm_Vertical, symbol Connector:Conn_01x01_Pin
- added C1, C2, C3, C4, C5, C6, C7, C8, C9: 100nF, symbol LoRa_Boat_Controller:C
- added C10, CEXT: 4.7uF, symbol LoRa_Boat_Controller:C
- added C12, C22: 0.1uF, symbol LoRa_Boat_Controller:C
- added C14: 470pF, symbol LoRa_Boat_Controller:C
- added C20, C21, CIN, COUT: 10uF, symbol LoRa_Boat_Controller:C
- added C23: 47pF, symbol LoRa_Boat_Controller:C
- added CANHEADER: B4B-XH-A, symbol LoRa_Boat_Controller:Conn_01x04_JST
- added D21: CMS06TE12L, symbol LoRa_Boat_Controller:SB007_03Q
- added GND_J: Battery-, symbol LoRa_Boat_Controller:Conn_01x01
- added GPSMODULE: NEO-6M, symbol LoRa_Boat_Controller:Conn_01x05
- added JTAG: FTSH-105, symbol LoRa_Boat_Controller:Conn_02x05_JTAG
- added L1: 4.7uH, symbol LoRa_Boat_Controller:L
- added L3, L4: Ferrite, symbol LoRa_Boat_Controller:L
- added LORAMODULE: RYLR896, symbol LoRa_Boat_Controller:Conn_01x05
- added R1: 15K, symbol LoRa_Boat_Controller:R
- added R2: 4.7K, symbol LoRa_Boat_Controller:R
- added R3: 51, symbol LoRa_Boat_Controller:R
- added R4: 5.1K, symbol LoRa_Boat_Controller:R
- added R5: 30K, symbol LoRa_Boat_Controller:R
- added R6: 10K, symbol LoRa_Boat_Controller:R
- added SPEEDCONTROLLER: ESC_PWM, symbol LoRa_Boat_Controller:Conn_01x03
- added STEERINGSERVO: RUDDER_PWM, symbol LoRa_Boat_Controller:Conn_01x03
- added TP1: PWM_MOT, symbol LoRa_Boat_Controller:TestPoint
- added TP3: PWM_RUD, symbol LoRa_Boat_Controller:TestPoint
- added TP4: 3V3_OUT, symbol LoRa_Boat_Controller:TestPoint
- added TP5: GND_TP, symbol LoRa_Boat_Controller:TestPoint
- added U3: STM32F446RET6, symbol LoRa_Boat_Controller:STM32F446RETx
- added U5: TCAN1042HDRQ1, symbol LoRa_Boat_Controller:TCAN1042H_Q1
- added U6: R1240N001B, symbol LoRa_Boat_Controller:R1240N001x
- added VIN: Battery+, symbol LoRa_Boat_Controller:Conn_01x01
- added _TEMPLATE_C: C_TEMPLATE, symbol Device:C
- added _TEMPLATE_D: LED_TEMPLATE, symbol Device:LED
- added _TEMPLATE_R: R_TEMPLATE, symbol Device:R
Other:
- note removed: "CAN Bus Transceiver"
- note removed: "Debug / JTAG"
- note removed: "GPS Module"
- note removed: "LoRa Module (RYLR)"
- note removed: "MCU - STM32F446RET6"
- note removed: "PWM Outputs"
- note removed: "Power Supply"
- title: LoRa Autonomous Boat Controller -> (none)

Commit message: Phase A3: hierarchical V1 schematic generated from pstxnet.dat, ERC clean, netlist == pstxnet
gen_symbols.py (R1240N001x, TCAN1042H-Q1, CMS06 diode, VIN_RAW power symbol per current datasheets),
kicad_sym.py (flattened embedding of KiCad 9 library symbols), gen_sch.py (7 sub-sheets mirroring the OrCAD
blocks, labels/hierarchical pins/power symbols, deterministic symbol paths shared with the PCB via v1_design.py),
check_netlist.py (schematic and board nets == pstxnet.dat, refs and footprint paths match).
ERC 0 violations with --severity-all. Allegro refdes without a trailing digit get a '1' suffix (KiCad annotation
rule); original kept in the Allegro_RefDes property.

Co-Authored-By: Claude Fable 5.1 <noreply@anthropic.com>
Parts:
- removed C1, C2, C3, C4, C5, C6, C7, C8, C9: 100nF, symbol LoRa_Boat_Controller:C
- removed C10, CEXT: 4.7uF, symbol LoRa_Boat_Controller:C
- removed C12, C22: 0.1uF, symbol LoRa_Boat_Controller:C
- removed C14: 470pF, symbol LoRa_Boat_Controller:C
- removed C20, C21, CIN, COUT: 10uF, symbol LoRa_Boat_Controller:C
- removed C23: 47pF, symbol LoRa_Boat_Controller:C
- removed CANHEADER: B4B-XH-A, symbol LoRa_Boat_Controller:Conn_01x04_JST
- removed D21: CMS06TE12L, symbol LoRa_Boat_Controller:SB007_03Q
- removed GND_J: Battery-, symbol LoRa_Boat_Controller:Conn_01x01
- removed GPSMODULE: NEO-6M, symbol LoRa_Boat_Controller:Conn_01x05
- removed JTAG: FTSH-105, symbol LoRa_Boat_Controller:Conn_02x05_JTAG
- removed L1: 4.7uH, symbol LoRa_Boat_Controller:L
- removed L3, L4: Ferrite, symbol LoRa_Boat_Controller:L
- removed LORAMODULE: RYLR896, symbol LoRa_Boat_Controller:Conn_01x05
- removed R1: 15K, symbol LoRa_Boat_Controller:R
- removed R2: 4.7K, symbol LoRa_Boat_Controller:R
- removed R3: 51, symbol LoRa_Boat_Controller:R
- removed R4: 5.1K, symbol LoRa_Boat_Controller:R
- removed R5: 30K, symbol LoRa_Boat_Controller:R
- removed R6: 10K, symbol LoRa_Boat_Controller:R
- removed SPEEDCONTROLLER: ESC_PWM, symbol LoRa_Boat_Controller:Conn_01x03
- removed STEERINGSERVO: RUDDER_PWM, symbol LoRa_Boat_Controller:Conn_01x03
- removed TP1: PWM_MOT, symbol LoRa_Boat_Controller:TestPoint
- removed TP3: PWM_RUD, symbol LoRa_Boat_Controller:TestPoint
- removed TP4: 3V3_OUT, symbol LoRa_Boat_Controller:TestPoint
- removed TP5: GND_TP, symbol LoRa_Boat_Controller:TestPoint
- removed U3: STM32F446RET6, symbol LoRa_Boat_Controller:STM32F446RETx
- removed U5: TCAN1042HDRQ1, symbol LoRa_Boat_Controller:TCAN1042H_Q1
- removed U6: R1240N001B, symbol LoRa_Boat_Controller:R1240N001x
- removed VIN: Battery+, symbol LoRa_Boat_Controller:Conn_01x01
- removed _TEMPLATE_C: C_TEMPLATE, symbol Device:C
- removed _TEMPLATE_D: LED_TEMPLATE, symbol Device:LED
- removed _TEMPLATE_R: R_TEMPLATE, symbol Device:R
Other:
- added sheet CAN_Bus (CAN_Bus.kicad_sch)
- added sheet Debug (Debug.kicad_sch)
- added sheet GPS_Module (GPS_Module.kicad_sch)
- added sheet LoRa_Module (LoRa_Module.kicad_sch)
- added sheet MCU (MCU.kicad_sch)
- added sheet PWM_Outputs (PWM_Outputs.kicad_sch)
- added sheet PowerSupply (PowerSupply.kicad_sch)
- note added: "LoRa Autonomous Boat Controller V1 - as fabricated (senior design v5.brd, 2025-05-09). Hierarchy mirrors the OrCAD Capture blocks."
- note added: "OrCAD block: CANBUS module (TCAN1042H-Q1, C1, JST XH header; VCC supplied through the header)"
- note added: "OrCAD block: JTAG Header (Samtec FTSH-105, ARM 10-pin Cortex debug pinout)"
- note added: "OrCAD block: LORA Module (RYLR header, BLM15 ferrite pi-filter L3/L4 with C20-C23)"
- note added: "OrCAD blocks: MCU OUTPUTS + MCU power (STM32F446RET6, decoupling C2-C10, CEXT on VCAP_1)"
- note added: "OrCAD blocks: Power Supply / POWER BLOCK (battery pads, R1240N buck, D21 catch diode, VBAT divider, TP4/TP5)"
- note added: "OrCAD blocks: Speed Controller + Steering Servo headers (3V3 / signal / GND) with TP1, TP3"
- note added: "OrCAD: TOP VIEW (GPS 1x5 header: 3V3, GND, PB0, USART3_RX, USART3_TX)"
- note added: "Power rails GND, +3V3 and VIN_RAW are global power symbols; every other inter-sheet net enters through the sheet pins below."
- company: (none) -> University of Arkansas EECS
- title: (none) -> LoRa Autonomous Boat Controller V1 - Root
