File: hardware/kicad/Debug.kicad_sch (KiCad schematic)
At the start: 1 part

Commit message: Phase A3 close: CANH/CANL net names corrected, BOM with MPNs, DSN-v2 comparison, schematic exports
- gen_pcb.py: N04855 is CANL (U5 pin 6) and N24691 is CANH (U5 pin 7) per pstxnet.dat + TI SLLSES9D; the
  old NETLIST.md had them reversed (Codex review finding R03).
- gen_bom.py: docs/BOM.csv regenerated from the schematic with MPN/manufacturer/description/confidence/price
  columns (research in docs/research/BOM_MPN_RESEARCH.md, prices 2026-09-16).
- a0_xor_dsn.py: DSN v2 copper vs v5 films = 54 % / 63 % mismatch, 0 of 20 vias coincide, 0 of 45 parts unmoved;
  the DSN wiring is unusable for v5 (documented in docs/A0_PROVENANCE.md).
- Schematic PDF and per-sheet SVG exports in docs/img.
Gates: DRC 0 errors / 0 unconnected, ERC 0 violations, netlist check PASS, XOR F.Cu 0.87 % B.Cu 0.23 %.

Co-Authored-By: Claude Fable 5.1 <noreply@anthropic.com>
Parts:
- JTAG1: MPN (none) -> FTSH-105-01-L-DV-K; Manufacturer (none) -> Samtec
Changed lines of the file:
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@@
 			)
 		)
-		(property "Description" "Generic connector, double row, 02x05, odd/even pin numbering scheme (row 1 odd numbers, row 2 even numbers), script generated (kicad-library-utils/schlib/autogen/connector/)"
+		(property "Description" "2x5 1.27 mm SMT header, keyed (ARM Cortex 10-pin debug)"
 			(at 58.42 38.1 0)
 			(effects
@@
 			(at 58.42 38.1 0)
 			(effects
+				(font
+					(size 1.27 1.27)
+				)
+				(hide yes)
+			)
+		)
+		(property "MPN" "FTSH-105-01-L-DV-K"
+			(at 58.42 38.1 0)
+			(effects
+				(font
+					(size 1.27 1.27)
+				)
+				(hide yes)
+			)
+		)
+		(property "Manufacturer" "Samtec"
+			(at 58.42 38.1 0)
+			(effects
