File: hardware/kicad/MCU.kicad_sch (KiCad schematic)
At the start: 3 parts

Commit message: Phase A3: hierarchical V1 schematic generated from pstxnet.dat, ERC clean, netlist == pstxnet
gen_symbols.py (R1240N001x, TCAN1042H-Q1, CMS06 diode, VIN_RAW power symbol per current datasheets),
kicad_sym.py (flattened embedding of KiCad 9 library symbols), gen_sch.py (7 sub-sheets mirroring the OrCAD
blocks, labels/hierarchical pins/power symbols, deterministic symbol paths shared with the PCB via v1_design.py),
check_netlist.py (schematic and board nets == pstxnet.dat, refs and footprint paths match).
ERC 0 violations with --severity-all. Allegro refdes without a trailing digit get a '1' suffix (KiCad annotation
rule); original kept in the Allegro_RefDes property.

Co-Authored-By: Claude Fable 5.1 <noreply@anthropic.com>
Parts:
- removed _TEMPLATE_C: C_TEMPLATE, symbol Device:C
- removed _TEMPLATE_D: LED_TEMPLATE, symbol Device:LED
- removed _TEMPLATE_R: R_TEMPLATE, symbol Device:R
- added C10, CEXT1: 4.7uF, LoRa_Boat_Controller:CAP_0603_CL10A_1P6XP8_SAM-M, symbol Device:C
- added C2, C3, C4, C5, C6, C7, C8, C9: 1uF, LoRa_Boat_Controller:CAP_KGM21_KAV-L, symbol Device:C
- added U3: STM32F446RET6, LoRa_Boat_Controller:LQFP64-10x10mm, symbol MCU_ST_STM32F4:STM32F446RETx
Connections:
- new net +3V3: C10.2, C2.2, C3.2, C4.2, C5.2, C6.2, C7.2, C8.2, C9.2, CEXT1.2, U3.13 (VDDA), U3.19 (VDD), U3.32 (VDD), U3.48 (VDD), U3.64 (VDD)
- new net ADC_VBAT: U3.16 (PA2)
- new net CAN_RXD_PA10: U3.43 (PA10)
- new net CAN_STB_PA11: U3.44 (PA11)
- new net CAN_TXD_PA12: U3.45 (PA12)
- new net GND: C10.1, C2.1, C3.1, C4.1, C5.1, C6.1, C7.1, C8.1, C9.1, U3.12 (VSSA), U3.18 (VSS), U3.31 (VSS), U3.47 (VSS), U3.63 (VSS)
- new net GPS_PB0: U3.26 (PB0)
- new net GPS_RX_PC11: U3.52 (PC11)
- new net GPS_TX_PC10: U3.51 (PC10)
- new net LORA_RST_PA3: U3.17 (PA3)
- new net LORA_RX_PA1: U3.15 (PA1)
- new net LORA_TX_PA0: U3.14 (PA0)
- new net NRST: U3.7 (NRST)
- new net PWM_PA8_ESCHDR: U3.41 (PA8)
- new net PWM_PC6_SERVOHDR: U3.37 (PC6)
- new net SWCLK: U3.49 (PA14)
- new net SWDIO: U3.46 (PA13)
- new net SWO_TDO: U3.55 (PB3)
- new net TDI: U3.50 (PA15)
- new net VCAP1: CEXT1.1, U3.30 (VCAP_1)
- no-connect marks 0 -> 36
Other:
- note added: "Allegro net names: +3V3<-3.3V, ADC_VBAT<-ADC, CAN_RXD_PA10<-N04759, CAN_STB_PA11<-N04755, CAN_TXD_PA12<-N04763, GND<-0, GPS_PB0<-N04277, GPS_RX_PC11<-N04281, GPS_TX_PC10<-N04285, LORA_RST_PA3<-N24517, LORA_RX_PA1<-N04485, LORA_TX_PA0<-N04477, NRST<-RESET, PWM_PA8_ESCHDR<-N04355, PWM_PC6_SERVOHDR<-N04395, SWCLK<-PA14 TCLK, SWDIO<-PA13 TMS, SWO_TDO<-PB3 TBO, TDI<-PA15 TDI, VCAP1<-N27791"
- note added: "MCU: OrCAD blocks: MCU OUTPUTS + MCU power (STM32F446RET6, decoupling C2-C10, CEXT on VCAP_1)"
- note added: "VBAT (pin 1) is unconnected on the fabricated board (single-node net in pstxnet.dat); BOOT0 (pin 60) is unconnected."
- company: (none) -> University of Arkansas EECS
- title: (none) -> LoRa Autonomous Boat Controller V1 - MCU

Commit message: Phase A3 close: CANH/CANL net names corrected, BOM with MPNs, DSN-v2 comparison, schematic exports
- gen_pcb.py: N04855 is CANL (U5 pin 6) and N24691 is CANH (U5 pin 7) per pstxnet.dat + TI SLLSES9D; the
  old NETLIST.md had them reversed (Codex review finding R03).
- gen_bom.py: docs/BOM.csv regenerated from the schematic with MPN/manufacturer/description/confidence/price
  columns (research in docs/research/BOM_MPN_RESEARCH.md, prices 2026-09-16).
- a0_xor_dsn.py: DSN v2 copper vs v5 films = 54 % / 63 % mismatch, 0 of 20 vias coincide, 0 of 45 parts unmoved;
  the DSN wiring is unusable for v5 (documented in docs/A0_PROVENANCE.md).
- Schematic PDF and per-sheet SVG exports in docs/img.
Gates: DRC 0 errors / 0 unconnected, ERC 0 violations, netlist check PASS, XOR F.Cu 0.87 % B.Cu 0.23 %.

Co-Authored-By: Claude Fable 5.1 <noreply@anthropic.com>
Parts:
- C10, CEXT1: MPN (none) -> CL10A475KP8NNNC; Manufacturer (none) -> Samsung Electro-Mechanics
- C2, C3, C4, C5, C6, C7, C8, C9: value 1uF -> 0.1uF; MPN (none) -> KGM21NR71H104KT; Manufacturer (none) -> Kyocera AVX
- U3: MPN (none) -> STM32F446RET6; Manufacturer (none) -> STMicroelectronics
Changed lines of the file:
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@@
 			)
 		)
-		(property "Description" "STMicroelectronics Arm Cortex-M4 MCU, 512KB flash, 128KB RAM, 180 MHz, 1.8-3.6V, 50 GPIO, LQFP64"
+		(property "Description" "Arm Cortex-M4 180 MHz, 512 KB flash, 128 KB SRAM, LQFP-64 (TR = tape-and-reel of the same die)"
 			(at 73.66 81.28 0)
 			(effects
@@
 		)
 		(property "Allegro_Device" "STM32F446RET6TR_LQFP64-10X10MM_STM32F4XXR2"
+			(at 73.66 81.28 0)
+			(effects
+				(font
+					(size 1.27 1.27)
+				)
+				(hide yes)
+			)
+		)
+		(property "MPN" "STM32F446RET6"
+			(at 73.66 81.28 0)
+			(effects
+				(font
+					(size 1.27 1.27)
+				)
+				(hide yes)
+			)
+		)
+		(property "Manufacturer" "STMicroelectronics"
 			(at 73.66 81.28 0)
 			(effects
@@
 			)
 		)
-		(property "Description" "Unpolarized capacitor"
+		(property "Description" "4.7 uF 10% 10 V X5R MLCC 0603 (design gives CL10A + 0603 only; 10 V chosen)"
 			(at 134.62 35.56 0)
 			(effects
@@
 		)
 		(property "Allegro_Device" "C_CAP_0603_CL10A_1P6XP8_SAM-M_4.7 UF"
+			(at 134.62 35.56 0)
+			(effects
+				(font
+					(size 1.27 1.27)
+				)
+				(hide yes)
+			)
+		)
+		(property "MPN" "CL10A475KP8NNNC"
+			(at 134.62 35.56 0)
+			(effects
+				(font
+					(size 1.27 1.27)
+				)
+				(hide yes)
+			)
+		)
+		(property "Manufacturer" "Samsung Electro-Mechanics"
 			(at 134.62 35.56 0)
 			(effects
@@
 			)
 		)
-		(property "Description" "Unpolarized capacitor"
+		(property "Description" "4.7 uF 10% 10 V X5R MLCC 0603 (design gives CL10A + 0603 only; 10 V chosen)"
 			(at 180.34 35.56 0)
 			(effects
@@
 			)
 		)
+		(property "MPN" "CL10A475KP8NNNC"
+			(at 180.34 35.56 0)
+			(effects
+				(font
+					(size 1.27 1.27)
+				)
+				(hide yes)
+			)
+		)
+		(property "Manufacturer" "Samsung Electro-Mechanics"
+			(at 180.34 35.56 0)
+			(effects
+				(font
+					(size 1.27 1.27)
+				)
+				(hide yes)
+			)
+		)
 		(property "Allegro_RefDes" "C10"
 			(at 180.34 35.56 0)
@@
 			)
 		)
-		(property "Value" "1uF"
+		(property "Value" "0.1uF"
 			(at 223.52 40.87 0)
 			(effects
@@
 			)
 		)
-		(property "Description" "Unpolarized capacitor"
+		(property "Description" "0.1 uF 10% 50 V X7R MLCC 0805"
 			(at 223.52 35.56 0)
 			(effects
@@
 			)
 		)
+		(property "MPN" "KGM21NR71H104KT"
+			(at 223.52 35.56 0)
+			(effects
+				(font
+					(size 1.27 1.27)
+				)
+				(hide yes)
+			)
+		)
+		(property "Manufacturer" "Kyocera AVX"
+			(at 223.52 35.56 0)
+			(effects
+				(font
+					(size 1.27 1.27)
+				)
+				(hide yes)
+			)
+		)
 		(property "Allegro_RefDes" "C2"
 			(at 223.52 35.56 0)
@@
 			)
 		)
-		(property "Value" "1uF"
+		(property "Value" "0.1uF"
 			(at 266.7 40.87 0)
 			(effects
@@
 			)
 		)
-		(property "Description" "Unpolarized capacitor"
+		(property "Description" "0.1 uF 10% 50 V X7R MLCC 0805"
 			(at 266.7 35.56 0)
 			(effects
@@
 			)
 		)
+		(property "MPN" "KGM21NR71H104KT"
+			(at 266.7 35.56 0)
+			(effects
+				(font
+					(size 1.27 1.27)
+				)
+				(hide yes)
+			)
+		)
+		(property "Manufacturer" "Kyocera AVX"
+			(at 266.7 35.56 0)
+			(effects
+				(font
+					(size 1.27 1.27)
+				)
+				(hide yes)
+			)
+		)
 		(property "Allegro_RefDes" "C3"
 			(at 266.7 35.56 0)
@@
 			)
 		)
-		(property "Value" "1uF"
+		(property "Value" "0.1uF"
 			(at 312.42 40.87 0)
 			(effects
@@
 			)
 		)
-		(property "Description" "Unpolarized capacitor"
+		(property "Description" "0.1 uF 10% 50 V X7R MLCC 0805"
 			(at 312.42 35.56 0)
 			(effects
@@
 			)
 		)
+		(property "MPN" "KGM21NR71H104KT"
+			(at 312.42 35.56 0)
+			(effects
+				(font
+					(size 1.27 1.27)
+				)
+				(hide yes)
+			)
+		)
+		(property "Manufacturer" "Kyocera AVX"
+			(at 312.42 35.56 0)
+			(effects
+				(font
+					(size 1.27 1.27)
+				)
+				(hide yes)
+			)
+		)
 		(property "Allegro_RefDes" "C4"
 			(at 312.42 35.56 0)
@@
 			)
 		)
-		(property "Value" "1uF"
+		(property "Value" "0.1uF"
 			(at 355.6 40.87 0)
 			(effects
@@
 			)
 		)
-		(property "Description" "Unpolarized capacitor"
+		(property "Description" "0.1 uF 10% 50 V X7R MLCC 0805"
 			(at 355.6 35.56 0)
 			(effects
@@
 			)
 		)
+		(property "MPN" "KGM21NR71H104KT"
+			(at 355.6 35.56 0)
+			(effects
+				(font
+					(size 1.27 1.27)
+				)
+				(hide yes)
+			)
+		)
+		(property "Manufacturer" "Kyocera AVX"
+			(at 355.6 35.56 0)
+			(effects
+				(font
+					(size 1.27 1.27)
+				)
+				(hide yes)
+			)
+		)
 		(property "Allegro_RefDes" "C5"
 			(at 355.6 35.56 0)
@@
 			)
 		)
-		(property "Value" "1uF"
+		(property "Value" "0.1uF"
 			(at 55.88 150.09 0)
 			(effects
@@
 			)
 		)
-		(property "Description" "Unpolarized capacitor"
+		(property "Description" "0.1 uF 10% 50 V X7R MLCC 0805"
 			(at 55.88 144.78 0)
 			(effects
@@
 			)
 		)
+		(property "MPN" "KGM21NR71H104KT"
+			(at 55.88 144.78 0)
+			(effects
+				(font
+					(size 1.27 1.27)
+				)
+				(hide yes)
+			)
+		)
+		(property "Manufacturer" "Kyocera AVX"
+			(at 55.88 144.78 0)
+			(effects
+				(font
+					(size 1.27 1.27)
+				)
+				(hide yes)
+			)
+		)
 		(property "Allegro_RefDes" "C6"
 			(at 55.88 144.78 0)
@@
 			)
 		)
-		(property "Value" "1uF"
+		(property "Value" "0.1uF"
 			(at 99.06 150.09 0)
 			(effects
@@
 			)
 		)
-		(property "Description" "Unpolarized capacitor"
+		(property "Description" "0.1 uF 10% 50 V X7R MLCC 0805"
 			(at 99.06 144.78 0)
 			(effects
@@
 			)
 		)
+		(property "MPN" "KGM21NR71H104KT"
+			(at 99.06 144.78 0)
+			(effects
+				(font
+					(size 1.27 1.27)
+				)
+				(hide yes)
+			)
+		)
+		(property "Manufacturer" "Kyocera AVX"
+			(at 99.06 144.78 0)
+			(effects
+				(font
+					(size 1.27 1.27)
+				)
+				(hide yes)
+			)
+		)
 		(property "Allegro_RefDes" "C7"
 			(at 99.06 144.78 0)
@@
 			)
 		)
-		(property "Value" "1uF"
+		(property "Value" "0.1uF"
 			(at 142.24 150.09 0)
 			(effects
@@
 			)
 		)
-		(property "Description" "Unpolarized capacitor"
+		(property "Description" "0.1 uF 10% 50 V X7R MLCC 0805"
 			(at 142.24 144.78 0)
 			(effects
@@
 			)
 		)
+		(property "MPN" "KGM21NR71H104KT"
+			(at 142.24 144.78 0)
+			(effects
+				(font
+					(size 1.27 1.27)
+				)
+				(hide yes)
+			)
+		)
+		(property "Manufacturer" "Kyocera AVX"
+			(at 142.24 144.78 0)
+			(effects
+				(font
+					(size 1.27 1.27)
+				)
+				(hide yes)
+			)
+		)
 		(property "Allegro_RefDes" "C8"
 			(at 142.24 144.78 0)
@@
 			)
 		)
-		(property "Value" "1uF"
+		(property "Value" "0.1uF"
 			(at 187.96 150.09 0)
 			(effects
@@
 			)
 		)
-		(property "Description" "Unpolarized capacitor"
+		(property "Description" "0.1 uF 10% 50 V X7R MLCC 0805"
 			(at 187.96 144.78 0)
 			(effects
@@
 			(at 187.96 144.78 0)
 			(effects
+				(font
+					(size 1.27 1.27)
+				)
+				(hide yes)
+			)
+		)
+		(property "MPN" "KGM21NR71H104KT"
+			(at 187.96 144.78 0)
+			(effects
+				(font
+					(size 1.27 1.27)
+				)
+				(hide yes)
+			)
+		)
+		(property "Manufacturer" "Kyocera AVX"
+			(at 187.96 144.78 0)
+			(effects
