File: hardware/kicad_v2/Debug.kicad_sch (KiCad schematic)
At the start: 7 parts, among them J6 USB-C, J7 SWD, U7 USBLC6-2SC6

Commit message: Phase C draft closed: GND stitch pass, review fixes (U3 no-connect, D2 10 V, VBUS divider), renders, docs index, release notes
- route_v2.py: isolated GND clusters found by union-find over the filled pour outlines (joined through vias and THT pads),
  stitched with straight or L-shaped 0.25 mm tracks to the connected pour, accepted only when the unconnected count drops;
  1 of 3 islands stitched on this layout, 2 remain for hand-finish (documented in hardware/kicad_v2/README.md and REPORT.md)
- gen_v2.py: V2 no longer inherits the V1 FORCE_NC (TPS54202 pin 1 had a no-connect flag in the schematic); GND pours solid-connected
- v2_design.py: D2 BZT52C10 (10 V clamp, AO3401A Vgs max 12 V), R28 47k (PA9 sees 2.5 V), BOM 67 lines $53.80
- board: 1075 segments, 165 vias, DRC 0 violations, 2 unconnected; renders docs/img/v2_pcb_top/bottom.png, copper SVGs
- REPORT.md numbers filled in (35 V1 findings, routing stats); BLOCKERS decision-7 row updated; docs/INDEX.md regenerated with V2 entries;
  HANDOFF/AGENT_STATUS release note; CONVERSION_LOG entry

Co-Authored-By: Claude Fable 5.1 <noreply@anthropic.com>
Parts:
- R28: value 22k -> 47k; MPN RC0603FR-0722KL -> RC0603FR-0747KL
Changed lines of the file:
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@@
 			)
 		)
-		(property "Value" "22k"
+		(property "Value" "47k"
 			(at 53.34 96.75 0)
 			(effects
@@
 			)
 		)
-		(property "Description" "VBUS sense bottom (5 V -> 1.6 V on PA9)"
+		(property "Description" "VBUS sense bottom (5 V -> 2.5 V on PA9 as a plain GPIO/ADC input, review A-12)"
 			(at 53.34 91.44 0)
 			(effects
@@
 			)
 		)
-		(property "MPN" "RC0603FR-0722KL"
+		(property "MPN" "RC0603FR-0747KL"
 			(at 53.34 91.44 0)
 			(effects
