File: hardware/kicad_v2/Power.kicad_sch (KiCad schematic)
At the start: 42 parts, among them J1 BATTERY XT30, Q1 AO3401A, U2 R1240N001B-TR-FE, U3 TPS54202, U8 INA180A1

Commit message: Phase C draft closed: GND stitch pass, review fixes (U3 no-connect, D2 10 V, VBUS divider), renders, docs index, release notes
- route_v2.py: isolated GND clusters found by union-find over the filled pour outlines (joined through vias and THT pads),
  stitched with straight or L-shaped 0.25 mm tracks to the connected pour, accepted only when the unconnected count drops;
  1 of 3 islands stitched on this layout, 2 remain for hand-finish (documented in hardware/kicad_v2/README.md and REPORT.md)
- gen_v2.py: V2 no longer inherits the V1 FORCE_NC (TPS54202 pin 1 had a no-connect flag in the schematic); GND pours solid-connected
- v2_design.py: D2 BZT52C10 (10 V clamp, AO3401A Vgs max 12 V), R28 47k (PA9 sees 2.5 V), BOM 67 lines $53.80
- board: 1075 segments, 165 vias, DRC 0 violations, 2 unconnected; renders docs/img/v2_pcb_top/bottom.png, copper SVGs
- REPORT.md numbers filled in (35 V1 findings, routing stats); BLOCKERS decision-7 row updated; docs/INDEX.md regenerated with V2 entries;
  HANDOFF/AGENT_STATUS release note; CONVERSION_LOG entry

Co-Authored-By: Claude Fable 5.1 <noreply@anthropic.com>
Parts:
- D2: value 12V -> 10V; MPN BZT52C12-7-F -> BZT52C10-7-F
Connections:
- net GND: now also U3.1 (GND)
- no-connect marks 1 -> 0
Changed lines of the file:
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@@
 			)
 		)
-		(property "Value" "12V"
+		(property "Value" "10V"
 			(at 193.04 35.79 0)
 			(effects
@@
 			)
 		)
-		(property "Description" "Gate-source clamp for Q1"
+		(property "Description" "Gate-source clamp for Q1 (10 V: AO3401A Vgs max is 12 V, review A-10)"
 			(at 193.04 33.02 0)
 			(effects
@@
 			)
 		)
-		(property "MPN" "BZT52C12-7-F"
+		(property "MPN" "BZT52C10-7-F"
 			(at 193.04 33.02 0)
 			(effects
@@
 		)
 	)
-	(no_connect
-		(at 106.68 127)
+	(wire
+		(pts
+			(xy 106.68 127) (xy 106.68 129.54)
+		)
+		(stroke
+			(width 0)
+			(type default)
+		)
+	)
+	(symbol
+		(lib_id "power:GND")
+		(at 106.68 129.54 0)
+		(unit 1)
+		(exclude_from_sim no)
+		(in_bom no)
+		(on_board no)
+		(dnp no)
+		(property "Reference" "#PWRPOW23"
+			(at 106.68 125.73 0)
+			(effects
+				(font
+					(size 1.27 1.27)
+				)
+			(hide yes)
+			)
+		)
+		(property "Value" "GND"
+			(at 106.68 133.096 0)
+			(effects
+				(font
+					(size 1.27 1.27)
+				)
+			)
+		)
+		(pin "1"
+		)
+		(instances
+			(project "LoRa_Boat_Controller_V2"
+				(path "/1dd45446-4f65-56e8-a2d3-9539c2076706/ab044879-1b8a-5671-848c-dc324c91f865"
+					(reference "#PWRPOW23")
+					(unit 1)
+				)
+			)
+		)
 	)
 	(wire
@@
 		(on_board no)
 		(dnp no)
-		(property "Reference" "#PWRPOW23"
+		(property "Reference" "#PWRPOW24"
 			(at 325.12 119.38 0)
 			(effects
@@
 			(project "LoRa_Boat_Controller_V2"
 				(path "/1dd45446-4f65-56e8-a2d3-9539c2076706/ab044879-1b8a-5671-848c-dc324c91f865"
-					(reference "#PWRPOW23")
+					(reference "#PWRPOW24")
 					(unit 1)
 				)
@@
 		(on_board no)
 		(dnp no)
-		(property "Reference" "#PWRPOW24"
+		(property "Reference" "#PWRPOW25"
 			(at 368.3 119.38 0)
 			(effects
@@
 			(project "LoRa_Boat_Controller_V2"
 				(path "/1dd45446-4f65-56e8-a2d3-9539c2076706/ab044879-1b8a-5671-848c-dc324c91f865"
-					(reference "#PWRPOW24")
+					(reference "#PWRPOW25")
 					(unit 1)
 				)
@@
 		(on_board no)
 		(dnp no)
-		(property "Reference" "#PWRPOW25"
+		(property "Reference" "#PWRPOW26"
 			(at 55.88 147.32 0)
 			(effects
@@
 			(project "LoRa_Boat_Controller_V2"
 				(path "/1dd45446-4f65-56e8-a2d3-9539c2076706/ab044879-1b8a-5671-848c-dc324c91f865"
-					(reference "#PWRPOW25")
+					(reference "#PWRPOW26")
 					(unit 1)
 				)
@@
 		(on_board no)
 		(dnp no)
-		(property "Reference" "#PWRPOW26"
+		(property "Reference" "#PWRPOW27"
 			(at 99.06 147.32 0)
 			(effects
@@
 			(project "LoRa_Boat_Controller_V2"
 				(path "/1dd45446-4f65-56e8-a2d3-9539c2076706/ab044879-1b8a-5671-848c-dc324c91f865"
-					(reference "#PWRPOW26")
+					(reference "#PWRPOW27")
 					(unit 1)
 				)
@@
 		(on_board no)
 		(dnp no)
-		(property "Reference" "#PWRPOW27"
+		(property "Reference" "#PWRPOW28"
 			(at 238.76 134.62 0)
 			(effects
@@
 			(project "LoRa_Boat_Controller_V2"
 				(path "/1dd45446-4f65-56e8-a2d3-9539c2076706/ab044879-1b8a-5671-848c-dc324c91f865"
-					(reference "#PWRPOW27")
+					(reference "#PWRPOW28")
 					(unit 1)
 				)
@@
 		(on_board no)
 		(dnp no)
-		(property "Reference" "#PWRPOW28"
+		(property "Reference" "#PWRPOW29"
 			(at 238.76 147.32 0)
 			(effects
@@
 			(project "LoRa_Boat_Controller_V2"
 				(path "/1dd45446-4f65-56e8-a2d3-9539c2076706/ab044879-1b8a-5671-848c-dc324c91f865"
-					(reference "#PWRPOW28")
+					(reference "#PWRPOW29")
 					(unit 1)
 				)
@@
 		(on_board no)
 		(dnp no)
-		(property "Reference" "#PWRPOW29"
+		(property "Reference" "#PWRPOW30"
 			(at 281.94 134.62 0)
 			(effects
@@
 			(project "LoRa_Boat_Controller_V2"
 				(path "/1dd45446-4f65-56e8-a2d3-9539c2076706/ab044879-1b8a-5671-848c-dc324c91f865"
-					(reference "#PWRPOW29")
+					(reference "#PWRPOW30")
 					(unit 1)
 				)
@@
 		(on_board no)
 		(dnp no)
-		(property "Reference" "#PWRPOW30"
+		(property "Reference" "#PWRPOW31"
 			(at 281.94 147.32 0)
 			(effects
@@
 			(project "LoRa_Boat_Controller_V2"
 				(path "/1dd45446-4f65-56e8-a2d3-9539c2076706/ab044879-1b8a-5671-848c-dc324c91f865"
-					(reference "#PWRPOW30")
+					(reference "#PWRPOW31")
 					(unit 1)
 				)
@@
 		(on_board no)
 		(dnp no)
-		(property "Reference" "#PWRPOW31"
+		(property "Reference" "#PWRPOW32"
 			(at 325.12 140.97 0)
 			(effects
@@
 			(project "LoRa_Boat_Controller_V2"
 				(path "/1dd45446-4f65-56e8-a2d3-9539c2076706/ab044879-1b8a-5671-848c-dc324c91f865"
-					(reference "#PWRPOW31")
+					(reference "#PWRPOW32")
 					(unit 1)
 				)
@@
 		(on_board no)
 		(dnp no)
-		(property "Reference" "#PWRPOW32"
+		(property "Reference" "#PWRPOW33"
 			(at 365.76 140.97 0)
 			(effects
@@
 			(project "LoRa_Boat_Controller_V2"
 				(path "/1dd45446-4f65-56e8-a2d3-9539c2076706/ab044879-1b8a-5671-848c-dc324c91f865"
-					(reference "#PWRPOW32")
+					(reference "#PWRPOW33")
 					(unit 1)
 				)
@@
 		(on_board no)
 		(dnp no)
-		(property "Reference" "#PWRPOW33"
+		(property "Reference" "#PWRPOW34"
 			(at 53.34 163.83 0)
 			(effects
@@
 			(project "LoRa_Boat_Controller_V2"
 				(path "/1dd45446-4f65-56e8-a2d3-9539c2076706/ab044879-1b8a-5671-848c-dc324c91f865"
-					(reference "#PWRPOW33")
+					(reference "#PWRPOW34")
 					(unit 1)
 				)
@@
 		(on_board no)
 		(dnp no)
-		(property "Reference" "#PWRPOW34"
+		(property "Reference" "#PWRPOW35"
 			(at 91.44 163.83 0)
 			(effects
@@
 			(project "LoRa_Boat_Controller_V2"
 				(path "/1dd45446-4f65-56e8-a2d3-9539c2076706/ab044879-1b8a-5671-848c-dc324c91f865"
-					(reference "#PWRPOW34")
+					(reference "#PWRPOW35")
 					(unit 1)
 				)
@@
 		(on_board no)
 		(dnp no)
-		(property "Reference" "#PWRPOW35"
+		(property "Reference" "#PWRPOW36"
 			(at 350.52 255.27 0)
 			(effects
@@
 			(project "LoRa_Boat_Controller_V2"
 				(path "/1dd45446-4f65-56e8-a2d3-9539c2076706/ab044879-1b8a-5671-848c-dc324c91f865"
-					(reference "#PWRPOW35")
+					(reference "#PWRPOW36")
 					(unit 1)
 				)
@@
 		(on_board no)
 		(dnp no)
-		(property "Reference" "#PWRPOW36"
+		(property "Reference" "#PWRPOW37"
 			(at 365.76 255.27 0)
 			(effects
@@
 			(project "LoRa_Boat_Controller_V2"
 				(path "/1dd45446-4f65-56e8-a2d3-9539c2076706/ab044879-1b8a-5671-848c-dc324c91f865"
-					(reference "#PWRPOW36")
+					(reference "#PWRPOW37")
 					(unit 1)
 				)
@@
 		(on_board no)
 		(dnp no)
-		(property "Reference" "#PWRPOW37"
+		(property "Reference" "#PWRPOW38"
 			(at 381 255.27 0)
 			(effects
@@
 			(project "LoRa_Boat_Controller_V2"
 				(path "/1dd45446-4f65-56e8-a2d3-9539c2076706/ab044879-1b8a-5671-848c-dc324c91f865"
-					(reference "#PWRPOW37")
+					(reference "#PWRPOW38")
 					(unit 1)
 				)
@@
 		(on_board no)
 		(dnp no)
-		(property "Reference" "#PWRPOW38"
+		(property "Reference" "#PWRPOW39"
 			(at 396.24 255.27 0)
 			(effects
@@
 			(project "LoRa_Boat_Controller_V2"
 				(path "/1dd45446-4f65-56e8-a2d3-9539c2076706/ab044879-1b8a-5671-848c-dc324c91f865"
-					(reference "#PWRPOW38")
+					(reference "#PWRPOW39")
 					(unit 1)
 				)
